Commit message: Update with xacro file

File: puma560_description/urdf/materials.xacro (robot description, xacro)
@@ -16,4 +16,7 @@
 		<color rgba="0.8 0.0 0.0 1.0"/>
 	</material>
+	<material name="red_transparent">
+		<color rgba="0.8 0.0 0.0 0.5"/>
+	</material>
 	<material name="white">
 		<color rgba="1.0 1.0 1.0 1.0"/>
