Commit message: Updated Puma model

File: puma560_description/urdf/puma560_v4.xacro (robot description, xacro)
@@ -3,177 +3,285 @@
 <robot name="puma560" xmlns:xacro="http://www.ros.org/wiki/xacro">
   <!-- Constants for robot dimensions -->
-  <xacro:property name="Pi" value="3.1415926535897931"/>
-  <!-- Geometric parameters for base-->
-  <xacro:property name="height_base" value="${.54864}"/>
-  <xacro:property name="mass" value="${0}"/>
-  <xacro:property name="com" value="${[0,0,0,0,0,0]}"/>
-  <xacro:property name="inertia_diagonals" value="${[0,0,0]}"/>
-  <xacro:property name="inertia_off_diagonal" value="${[0,0,0]}"/>
-  <xacro:macro name="general_inertia_defition" params="mass com inertia_diagonal inertia_off_diagonal">
-    <inertial>
-      <origin xyz="${com[1]} ${com[2]} ${com[3]}" rpy="${com[4]} ${com[5]} ${com[6]}"/>
-      <mass value="${mass}"/>
-      <inertia
-        ixx="${inertia_diagonal[1]}"  ixy="${inertia_off_diagonal[2]}" ixz="${inertia_off_diagonal[2]}"
-        iyy="${inertia_diagonal[2]}"  iyz="${inertia_off_diagonal[3]}"
-        izz="${inertia_diagonal[3]}"
-        />
-      </inertial>
-    </xacro:macro>
-    <!-- Import Rviz colors -->
-    <xacro:include filename="$(find puma560_description)/urdf/materials.xacro" />
-    <!-- Import all Gazebo-customization elements, including Gazebo colors -->
-    <xacro:include filename="$(find puma560_description)/urdf/puma560.gazebo" />
-    <!-- Link definitions -->
-    <link name="world"/>
-    <joint name="world" type="fixed">
-      <parent link="world"/>
-      <child link="puma_base"/>
-      <origin xyz="0 0 ${height_base}" rpy="0 0 0" />
-      <axis xyz="0 0 1" />
-    </joint>
-    <link name="puma_base">
-      <visual>
-        <origin xyz="0 0 0" rpy="0 0 0" />
-        <geometry>
-          <mesh filename="package://puma560_description/meshes/puma_base.stl" />
-        </geometry>
-        <material name="grey"/>
-      </visual>
-      <collision>
-        <origin xyz="0 0 0" rpy="0 0 0" />
-        <geometry>
-          <mesh filename="package://puma560_description/meshes/puma_base_collision.stl" />
-        </geometry>
-      </collision>
-</link>
-<!--      <xacro:general_inertia_defition
-        mass="42.62416"
-        com="[-0.000000, 0.021960, -0.356146, 0, 0, 0]"
-        inertia_diagonal="[1.48565, 1.36144, 0.43392]"
-        inertia_off_diagonal="[0, 0, 0.05984]"
-        />
-      </link>
-   <link name="puma_link_1">
+  <xacro:property name="Pi" value="${3.1415926535897931}"/>
+  <!-- Geometric parameters for base -->
+  <xacro:property name="offset_z_base" value="${0.54864}"/>
+  <xacro:property name="offset_z_link_1" value="${0.07493}"/>
+  <xacro:property name="offset_y_link_2" value="${0.14224 + 0.0254}"/>
+  <xacro:property name="offset_x_link_3" value="${0.4318}"/>
+  <xacro:property name="offset_x_link_4" value="${0.35179}"/>
+  <xacro:property name="offset_z_link_4" value="${0.0381}"/>
+  <xacro:property name="offset_z_link_5" value="${0.0803}"/>
+  <!-- Inertia parameters
+  mass and center of mass (com)
+  inertia_diagonal defined as [Ixx Iyy Izz]
+  inertia_off_diagonal defined as [Ixy Ixz Iyz]
+-->
+<xacro:macro name="general_inertia_definition" params="mass com inertia_diagonal inertia_off_diagonal">
+  <inertial>
+    <origin xyz="${com[0]} ${com[1]} ${com[2]}" rpy="${com[3]} ${com[4]} ${com[5]}"/>
+    <mass value="${mass}"/>
+    <inertia
+      ixx="${inertia_diagonal[0]}"
+      ixy="${inertia_off_diagonal[0]}"
+      ixz="${inertia_off_diagonal[1]}"
+      iyy="${inertia_diagonal[1]}"
+      iyz="${inertia_off_diagonal[2]}"
+      izz="${inertia_diagonal[2]}"
+      />
+    </inertial>
+  </xacro:macro>
+  <!-- Import Rviz colors -->
+  <xacro:include filename="$(find puma560_description)/urdf/materials.xacro" />
+  <!-- Import all Gazebo-customization elements, including Gazebo colors -->
+  <xacro:include filename="$(find puma560_description)/urdf/puma560.gazebo" />
+  <!-- Link definitions -->
+  <link name="world"/>
+  <joint name="world" type="fixed">
+    <parent link="world"/>
+    <child link="puma_base"/>
+    <origin xyz="0 0 ${offset_z_base}" rpy="0 0 0" />
+    <axis xyz="0 0 1" />
+  </joint>
+  <link name="puma_base">
     <visual>
-     <origin xyz="0 0 0" rpy="-${Pi/2} 0 -${Pi/2}" />
-     <geometry>
-      <mesh filename="package://puma560_description/meshes/puma_link_1.stl" />
-    </geometry>
-    <material name="metal"/>
-  </visual>
-  <inertial>
-    <origin xyz="0 0 0" rpy="0 0 0"/>
-    <mass value="${m_link_1}"/>
-    <inertia
-      ixx="${ixx_link_1}"   ixy="${ixy_link_1}"  ixz="${ixz_link_1}"
-      iyy="${iyy_link_1}"   iyz="${iyz_link_1}"
-      izz="${izz_link_1}"
-      />
-    </inertial>
-  </link>
-  <link name="puma_link_2">
-    <visual>
-      <origin xyz="0 0 0" rpy="${Pi} -${Pi/2} 0" />
+      <origin xyz="0 0 0" rpy="0 0 0" />
       <geometry>
-       <mesh filename="package://puma560_description/meshes/puma_link_2.stl" />
-     </geometry>
-     <material name="metal"/>
-   </visual>
-   <inertial>
-    <origin xyz="0 0 0" rpy="0 0 0"/>
-    <mass value="${m_link_2}"/>
-    <inertia
-      ixx="${ixx_link_2}"   ixy="${ixy_link_2}"  ixz="${ixz_link_2}"
-      iyy="${iyy_link_2}"   iyz="${iyz_link_2}"
-      izz="${izz_link_2}"
-      />
-    </inertial>
-  </link>
-  <link name="puma_link_3">
-    <visual>
-      <origin xyz="0 0 0" rpy="${Pi/2} -${Pi/2} 0 " />
-      <geometry>
-        <mesh filename="package://puma560_description/meshes/puma_link_3.stl" />
-      </geometry>
-      <material name="metal"/>
-    </visual>
-    <inertial>
-      <origin xyz="0 0 0" rpy="0 0 0"/>
-      <mass value="${m_link_3}"/>
-      <inertia
-        ixx="${ixx_link_3}"   ixy="${ixy_link_3}"  ixz="${ixz_link_3}"
-        iyy="${iyy_link_3}"   iyz="${iyz_link_3}"
-        izz="${izz_link_3}"
-        />
-      </inertial>
-    </link>
-    <link name="puma_link_4">
-      <visual>
-       <origin xyz="0 0 0" rpy="-${Pi/2} 0 0 " />
-       <geometry>
-        <mesh filename="package://puma560_description/meshes/puma_link_4.stl" />
+        <mesh filename="package://puma560_description/meshes/puma_base.stl" />
       </geometry>
       <material name="grey"/>
     </visual>
-    <inertial>
-      <origin xyz="0 0 0" rpy="0 0 0"/>
-      <mass value="${m_link_4}"/>
-      <inertia
-        ixx="${ixx_link_4}"   ixy="${ixy_link_4}"  ixz="${ixz_link_4}"
-        iyy="${iyy_link_4}"   iyz="${iyz_link_4}"
-        izz="${izz_link_4}"
-        />
-      </inertial>
-    </link>
-    <link name="puma_link_5">
-      <visual>
-       <origin xyz="0 0 0" rpy="0 ${Pi/2} 0 " />
-       <geometry>
-        <mesh filename="package://puma560_description/meshes/puma_link_5.stl" />
+    <collision>
+      <origin xyz="0 0 0" rpy="0 0 0" />
+      <geometry>
+        <mesh filename="package://puma560_description/meshes/puma_base_collision.stl" />
       </geometry>
-      <material name="grey"/>
-    </visual>
-    <inertial>
-      <origin xyz="0 0 0" rpy="0 0 0"/>
-      <mass value="${m_link_5}"/>
-      <inertia
-        ixx="${ixx_link_5}"   ixy="${ixy_link_5}"  ixz="${ixz_link_5}"
-        iyy="${iyy_link_5}"   iyz="${iyz_link_5}"
-        izz="${izz_link_5}"
-        />
-      </inertial>
-    </link> -->
-    <!-- Joint definitions -->
-<!--     <joint name="base_to_link_1" type="continuous">
-      <parent link="puma_base"/>
-      <child link="puma_link_1"/>
-      <origin xyz="0 0 0" rpy="0 0 0" />
-      <axis xyz="0 0 1" />
-    </joint>
-    <joint name="link_1_to_link_2" type="continuous">
-      <parent link="puma_link_1"/>
-      <child link="puma_link_2"/>
-      <origin xyz="0 ${d2} 0" rpy="${alpha1} 0 0" />
-      <axis xyz="0 0 1" />
-    </joint>
-    <joint name="link_2_to_link_3" type="continuous">
-      <parent link="puma_link_2"/>
-      <child link="puma_link_3"/>
-      <origin xyz="${a2} 0 0" rpy="0 0 0" />
-      <axis xyz="0 0 1" />
-    </joint>
-    <joint name="link_3_to_link_4" type="continuous">
-      <parent link="puma_link_3"/>
-      <child link="puma_link_4"/>
-      <origin xyz="${a3} 0 ${d3}" rpy="0 ${Pi/2} 0" />
-      <axis xyz="0 0 1" />
-    </joint>
-    <joint name="link_4_to_link_5" type="continuous">
-      <parent link="puma_link_4"/>
-      <child link="puma_link_5"/>
-      <origin xyz="0 0 ${d4}" rpy="${Pi/2} 0 0" />
-      <axis xyz="0 0 1" />
-    </joint>
-  -->
-</robot>
+    </collision>
+      <!-- Inertia parameters
+      mass and center of mass (com)
+      inertia_diagonal defined as [Ixx Iyy Izz]
+      inertia_off_diagonal defined as [Ixy Ixz Iyz]
+    -->
+    <!--     Parameters for uniform aluminium body -->
+    <xacro:general_inertia_definition
+      mass="42.62416"
+      com="${[-0.000000, 0.021960, -0.356146, 0, 0, 0]}"
+      inertia_diagonal="${[1.48565, 1.36144, 0.43392]}"
+      inertia_off_diagonal="${[0, 0, 0.05984]}"
+      />
+      <!--     Parameters for uniform generic body -->
+      <xacro:general_inertia_definition
+        mass="15.78673"
+        com="${[-0.000000, 0.021960, -0.356146, 0, 0, 0]}"
+        inertia_diagonal="${[0.55024, 0.50424, 0.16071]}"
+        inertia_off_diagonal="${[0, 0, 0.02216]}"
+        />
+      </link>
+      <joint name="link_1" type="continuous">
+        <parent link="puma_base"/>
+        <child link="puma_link_1"/>
+        <origin xyz="0 0 ${offset_z_link_1}" rpy="0 0 0" />
+        <axis xyz="0 0 1" />
+      </joint>
+      <link name="puma_link_1">
+        <visual>
+          <origin xyz="0 0 0" rpy="0 0 0" />
+          <geometry>
+            <mesh filename="package://puma560_description/meshes/puma_link_1.stl" />
+          </geometry>
+          <material name="metal"/>
+        </visual>
+        <collision>
+          <origin xyz="0 0 0" rpy="0 0 0" />
+          <geometry>
+            <mesh filename="package://puma560_description/meshes/puma_link_1_collision.stl" />
+          </geometry>
+        </collision>
+      <!-- Inertia parameters
+      mass and center of mass (com)
+      inertia_diagonal defined as [Ixx Iyy Izz]
+      inertia_off_diagonal defined as [Ixy Ixz Iyz]
+    -->
+    <!--     Parameters for uniform aluminium body -->
+    <xacro:general_inertia_definition
+      mass="11.97216"
+      com="${[-0.000000, 0.022503, -0.002794, 0, 0, 0]}"
+      inertia_diagonal="${[0.07379, 0.03595, 0.07334]}"
+      inertia_off_diagonal="${[0, 0, -0.00075]}"
+      />
+      <!--     Parameters for uniform generic body -->
+      <xacro:general_inertia_definition
+        mass="4.43413"
+        com="${[-0.000000, 0.022503, -0.002794, 0, 0, 0]}"
+        inertia_diagonal="${[0.02733, 0.01332, 0.02716]}"
+        inertia_off_diagonal="${[0, 0, -0.00028 ]}"
+        />
+      </link>
+      <joint name="link_2" type="continuous">
+        <parent link="puma_link_1"/>
+        <child link="puma_link_2"/>
+        <origin xyz="0 ${offset_y_link_2} 0" rpy="${Pi/2} 0 0" />
+        <axis xyz="0 0 1" />
+      </joint>
+      <link name="puma_link_2">
+        <visual>
+          <origin xyz="0 0 0" rpy="0 0 0" />
+          <geometry>
+            <mesh filename="package://puma560_description/meshes/puma_link_2.stl" />
+          </geometry>
+          <material name="metal"/>
+        </visual>
+        <collision>
+          <origin xyz="0 0 0" rpy="0 0 0" />
+          <geometry>
+            <mesh filename="package://puma560_description/meshes/puma_link_2_collision.stl" />
+          </geometry>
+        </collision>
+      <!-- Inertia parameters
+      mass and center of mass (com)
+      inertia_diagonal defined as [Ixx Iyy Izz]
+      inertia_off_diagonal defined as [Ixy Ixz Iyz]
+    -->
+    <!--     Parameters for uniform aluminium body -->
+    <xacro:general_inertia_definition
+      mass="45.48585"
+      com="${[0.082741, 0.000047, -0.047642, 0, 0, 0]}"
+      inertia_diagonal="${[0.26252, 1.61075, 1.78135]}"
+      inertia_off_diagonal="${[0.00002, 0.26252, -0.00013]}"
+      />
+      <!--     Parameters for uniform generic body -->
+      <xacro:general_inertia_definition
+        mass="16.84661"
+        com="${[0.082741, 0.000047, -0.047642, 0, 0, 0]}"
+        inertia_diagonal="${[0.09723, 0.59657, 0.65976]}"
+        inertia_off_diagonal="${[0.00001, 0.00435, -0.00005]}"
+        />
+      </link>
+      <joint name="link_3" type="continuous">
+        <parent link="puma_link_2"/>
+        <child link="puma_link_3"/>
+        <origin xyz="${offset_x_link_3} 0 0" rpy="0 0 0" />
+        <axis xyz="0 0 1" />
+      </joint>
+      <link name="puma_link_3">
+        <visual>
+          <origin xyz="0 0 0" rpy="0 0 0" />
+          <geometry>
+            <mesh filename="package://puma560_description/meshes/puma_link_3.stl" />
+          </geometry>
+          <material name="metal"/>
+        </visual>
+        <collision>
+          <origin xyz="0 0 0" rpy="0 0 0" />
+          <geometry>
+            <mesh filename="package://puma560_description/meshes/puma_link_3_collision.stl" />
+          </geometry>
+        </collision>
+      <!-- Inertia parameters
+      mass and center of mass (com)
+      inertia_diagonal defined as [Ixx Iyy Izz]
+      inertia_off_diagonal defined as [Ixy Ixz Iyz]
+    -->
+    <!--     Parameters for uniform aluminium body -->
+    <xacro:general_inertia_definition
+      mass="12.42678"
+      com="${[0.088782, -0.000001, 0.038098, 0, 0, 0]}"
+      inertia_diagonal="${[0.02482, 0.22306, 0.23586]}"
+      inertia_off_diagonal="${[0, 0, 0]}"
+      />
+      <!--     Parameters for uniform generic body -->
+      <xacro:general_inertia_definition
+        mass="4.60251"
+        com="${[0.088782, -0.000001, 0.038098, 0, 0, 0]}"
+        inertia_diagonal="${[0.00919, 0.08262, 0.08735]}"
+        inertia_off_diagonal="${[0, 0.00001, 0]}"
+        />
+      </link>
+      <joint name="link_4" type="continuous">
+        <parent link="puma_link_3"/>
+        <child link="puma_link_4"/>
+        <origin xyz="${offset_x_link_4} 0 ${offset_z_link_4} " rpy="0 ${Pi/2} 0" />
+        <axis xyz="0 0 1" />
+      </joint>
+      <link name="puma_link_4">
+        <visual>
+          <origin xyz="0 0 0" rpy="0 0 0" />
+          <geometry>
+            <mesh filename="package://puma560_description/meshes/puma_link_4.stl" />
+          </geometry>
+          <material name="orange"/>
+        </visual>
+        <collision>
+          <origin xyz="0 0 0" rpy="0 0 0" />
+          <geometry>
+            <mesh filename="package://puma560_description/meshes/puma_link_4_collision.stl" />
+          </geometry>
+        </collision>
+      <!-- Inertia parameters
+      mass and center of mass (com)
+      inertia_diagonal defined as [Ixx Iyy Izz]
+      inertia_off_diagonal defined as [Ixy Ixz Iyz]
+    -->
+    <!--     Parameters for uniform aluminium body -->
+    <xacro:general_inertia_definition
+      mass="1.27113"
+      com="${[-0.000000, -0.000000, 0.047887, 0, 0, 0]}"
+      inertia_diagonal="${[0.00209, 0.00199, 0.00126]}"
+      inertia_off_diagonal="${[0, 0, 0]}"
+      />
+      <!--     Parameters for uniform generic body -->
+    <xacro:general_inertia_definition
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