Commit message: Redefined urdf and added macro defition for inertia matrices

File: puma560_description/urdf/definitions.xacro (robot description, xacro)
@@ -1,5 +1,5 @@
 <?xml version="1.0"?>
 <robot name="puma560" xmlns:xacro="http://www.ros.org/wiki/xacro">
-  <!-- Inertia parameters
+  <!-- Create inertia matrix from parameters for general parts :
   mass[kg] and center of mass[m]
   inertia_diagonal defined as {Ixx Iyy Izz}[kg.m^2]
@@ -25,5 +25,5 @@
     </inertial>
   </xacro:macro>
-  <!-- Inertia parameters
+  <!-- Create inertia matrix from parameters for homogeneous parts :
   density[kg/m^3], volume[m^3] and center of mass[m]
   inertia_diagonal defined as {Ixx Iyy Izz}[m^4]
@@ -31,5 +31,5 @@
   -->
   <xacro:macro
-    name="homogeneous_inertia_definition_"
+    name="homogeneous_inertia_definition"
     params="density volume center_of_mass  inertia_diagonal inertia_off_diagonal">
   <inertial>

File: puma560_description/urdf/materials.xacro (robot description, xacro)
@@ -29,8 +29,8 @@
 	</material>
 	<material name="metal">
-		<color rgba="${211/255} ${211/255} ${211/255} 1" />
+		<color rgba="${211/255} ${211/255} ${211/255} 1.0" />
 	</material>
 	<material name="wood">
-		<color rgba="${205/255} ${133/255} ${63/255} 1" />
+		<color rgba="${205/255} ${133/255} ${63/255} 1.0" />
 	</material>
 </robot>

File: puma560_description/urdf/puma560.xacro (robot description, xacro)
@@ -2,7 +2,7 @@
 <!-- UNIMATE Puma 560 Manipulator -->
 <robot name="puma560" xmlns:xacro="http://www.ros.org/wiki/xacro">
-  <!-- Constants for robot dimensions -->
+  <!-- Some constants -->
   <xacro:property name="Pi" value="${3.1415926535897931}"/>
-  <!-- Geometric parameters for base -->
+  <!-- Geometric parameters for Puma 560-->
   <xacro:property name="offset_z_base" value="${0.54864}"/>
   <xacro:property name="offset_z_link_1" value="${0.07493}"/>
@@ -12,9 +12,27 @@
   <xacro:property name="offset_z_link_4" value="${0.0381}"/>
   <xacro:property name="offset_z_link_5" value="${0.0803}"/>
-  <!-- Import Rviz colors -->
+  <!-- Meshes location directory -->
+  <xacro:property name="mesh_path" value="package://puma560_description/meshes"/>
+  <!-- File suffix for collision parts -->
+  <xacro:property name="collision_suffix" value="_collision"/>
+  <!-- Visual mesh paths -->
+  <xacro:property name="puma_base_visual" value="${mesh_path}/puma_base.stl"/>
+  <xacro:property name="puma_link_1_visual" value="${mesh_path}/puma_link_1.stl"/>
+  <xacro:property name="puma_link_2_visual" value="${mesh_path}/puma_link_2.stl"/>
+  <xacro:property name="puma_link_3_visual" value="${mesh_path}/puma_link_3.stl"/>
+  <xacro:property name="puma_link_4_visual" value="${mesh_path}/puma_link_4.stl"/>
+  <xacro:property name="puma_link_5_visual" value="${mesh_path}/puma_link_5.stl"/>
+  <!-- Collsion mesh paths -->
+  <xacro:property name="puma_base_collision" value="${mesh_path}/puma_base${collision_suffix}.stl"/>
+  <xacro:property name="puma_link_1_collision" value="${mesh_path}/puma_link_1${collision_suffix}.stl"/>
+  <xacro:property name="puma_link_2_collision" value="${mesh_path}/puma_link_2${collision_suffix}.stl"/>
+  <xacro:property name="puma_link_3_collision" value="${mesh_path}/puma_link_3${collision_suffix}.stl"/>
+  <xacro:property name="puma_link_4_collision" value="${mesh_path}/puma_link_4${collision_suffix}.stl"/>
+  <xacro:property name="puma_link_5_collision" value="${mesh_path}/puma_link_5${collision_suffix}.stl"/>
+  <!-- Some esthetic color definitions -->
   <xacro:include filename="$(find puma560_description)/urdf/materials.xacro" />
-  <!-- Import xacro macro definition -->
+  <!-- Some xacro macro definitions -->
   <xacro:include filename="$(find puma560_description)/urdf/definitions.xacro" />
-  <!-- Import all Gazebo-customization elements, including Gazebo colors -->
+  <!-- Import Gazebo components for now colors and control plugin -->
   <xacro:include filename="$(find puma560_description)/urdf/puma560.gazebo" />
   <!-- Link definitions -->
@@ -30,5 +48,5 @@
       <origin xyz="0 0 0" rpy="0 0 0" />
       <geometry>
-        <mesh filename="package://puma560_description/meshes/puma_base.stl" />
+        <mesh filename="${puma_base_visual}" />
       </geometry>
       <material name="grey"/>
@@ -37,17 +55,15 @@
       <origin xyz="0 0 0" rpy="0 0 0" />
       <geometry>
-        <mesh filename="package://puma560_description/meshes/puma_base_collision.stl" />
+        <mesh filename="${puma_base_collision}" />
       </geometry>
     </collision>
-    <!--     Parameters for uniform aluminium body -->
-    <xacro:general_inertia_definition
-      mass="42.62416"
-      center_of_mass="${[-0.000000, 0.021960, -0.356146, 0, 0, 0]}"
-      inertia_diagonal="${[1.48565, 1.36144, 0.43392]}"
-      inertia_off_diagonal="${[0, 0, 0.05984]}"
-      />
-      <!--     Parameters for uniform generic body -->
-      <xacro:general_inertia_definition
-        mass="15.78673"
+      <!-- Create inertia matrix from parameters for homogeneous parts :
+      density[kg/m^3], volume[m^3] and center of mass[m]
+      inertia_diagonal defined as {Ixx Iyy Izz}[m^4]
+      inertia_off_diagonal defined as {Ixy Ixz Iyz}[m^4]
+      -->
+      <xacro:homogeneous_inertia_definition
+        density="1000"
+        volume="0.01578673"
         center_of_mass="${[-0.000000, 0.021960, -0.356146, 0, 0, 0]}"
         inertia_diagonal="${[0.55024, 0.50424, 0.16071]}"
@@ -65,5 +81,5 @@
           <origin xyz="0 0 0" rpy="0 0 0" />
           <geometry>
-            <mesh filename="package://puma560_description/meshes/puma_link_1.stl" />
+            <mesh filename="${puma_link_1_visual}" />
           </geometry>
           <material name="metal"/>
@@ -72,22 +88,15 @@
           <origin xyz="0 0 0" rpy="0 0 0" />
           <geometry>
-            <mesh filename="package://puma560_description/meshes/puma_link_1_collision.stl" />
-          </geometry>
-        </collision>
-      <!-- Inertia parameters
-      mass and center of mass (center_of_mass)
-      inertia_diagonal defined as [Ixx Iyy Izz]
-      inertia_off_diagonal defined as [Ixy Ixz Iyz]
-    -->
-    <!--     Parameters for uniform aluminium body -->
-    <xacro:general_inertia_definition
-      mass="11.97216"
-      center_of_mass="${[-0.000000, 0.022503, -0.002794, 0, 0, 0]}"
-      inertia_diagonal="${[0.07379, 0.03595, 0.07334]}"
-      inertia_off_diagonal="${[0, 0, -0.00075]}"
-      />
-      <!--     Parameters for uniform generic body -->
-      <xacro:general_inertia_definition
-        mass="4.43413"
+            <mesh filename="${puma_link_1_collision}" />
+          </geometry>
+        </collision>
+      <!-- Create inertia matrix from parameters for homogeneous parts :
+      density[kg/m^3], volume[m^3] and center of mass[m]
+      inertia_diagonal defined as {Ixx Iyy Izz}[m^4]
+      inertia_off_diagonal defined as {Ixy Ixz Iyz}[m^4]
+      -->
+      <xacro:homogeneous_inertia_definition
+        density="1000"
+        volume="0.00443413"
         center_of_mass="${[-0.000000, 0.022503, -0.002794, 0, 0, 0]}"
         inertia_diagonal="${[0.02733, 0.01332, 0.02716]}"
@@ -105,5 +114,5 @@
           <origin xyz="0 0 0" rpy="0 0 0" />
           <geometry>
-            <mesh filename="package://puma560_description/meshes/puma_link_2.stl" />
+            <mesh filename="${puma_link_2_visual}" />
           </geometry>
           <material name="metal"/>
@@ -112,22 +121,15 @@
           <origin xyz="0 0 0" rpy="0 0 0" />
           <geometry>
-            <mesh filename="package://puma560_description/meshes/puma_link_2_collision.stl" />
-          </geometry>
-        </collision>
-      <!-- Inertia parameters
-      mass and center of mass (center_of_mass)
-      inertia_diagonal defined as [Ixx Iyy Izz]
-      inertia_off_diagonal defined as [Ixy Ixz Iyz]
-    -->
-    <!--     Parameters for uniform aluminium body -->
-    <xacro:general_inertia_definition
-      mass="45.48585"
-      center_of_mass="${[0.082741, 0.000047, -0.047642, 0, 0, 0]}"
-      inertia_diagonal="${[0.26252, 1.61075, 1.78135]}"
-      inertia_off_diagonal="${[0.00002, 0.26252, -0.00013]}"
-      />
-      <!--     Parameters for uniform generic body -->
-      <xacro:general_inertia_definition
-        mass="16.84661"
+            <mesh filename="${puma_link_2_collision}" />
+          </geometry>
+        </collision>
+      <!-- Create inertia matrix from parameters for homogeneous parts :
+      density[kg/m^3], volume[m^3] and center of mass[m]
+      inertia_diagonal defined as {Ixx Iyy Izz}[m^4]
+      inertia_off_diagonal defined as {Ixy Ixz Iyz}[m^4]
+      -->
+      <xacro:homogeneous_inertia_definition
+        density="1000"
+        volume="0.01684661"
         center_of_mass="${[0.082741, 0.000047, -0.047642, 0, 0, 0]}"
         inertia_diagonal="${[0.09723, 0.59657, 0.65976]}"
@@ -145,5 +147,5 @@
           <origin xyz="0 0 0" rpy="0 0 0" />
           <geometry>
-            <mesh filename="package://puma560_description/meshes/puma_link_3.stl" />
+            <mesh filename="${puma_link_3_visual}" />
           </geometry>
           <material name="metal"/>
@@ -152,22 +154,15 @@
           <origin xyz="0 0 0" rpy="0 0 0" />
           <geometry>
-            <mesh filename="package://puma560_description/meshes/puma_link_3_collision.stl" />
-          </geometry>
-        </collision>
-      <!-- Inertia parameters
-      mass and center of mass (center_of_mass)
-      inertia_diagonal defined as [Ixx Iyy Izz]
-      inertia_off_diagonal defined as [Ixy Ixz Iyz]
-    -->
-    <!--     Parameters for uniform aluminium body -->
-    <xacro:general_inertia_definition
-      mass="12.42678"
-      center_of_mass="${[0.088782, -0.000001, 0.038098, 0, 0, 0]}"
-      inertia_diagonal="${[0.02482, 0.22306, 0.23586]}"
-      inertia_off_diagonal="${[0, 0, 0]}"
-      />
-      <!--     Parameters for uniform generic body -->
-      <xacro:general_inertia_definition
-        mass="4.60251"
+            <mesh filename="${puma_link_3_collision}" />
+          </geometry>
+        </collision>
+      <!-- Create inertia matrix from parameters for homogeneous parts :
+      density[kg/m^3], volume[m^3] and center of mass[m]
+      inertia_diagonal defined as {Ixx Iyy Izz}[m^4]
+      inertia_off_diagonal defined as {Ixy Ixz Iyz}[m^4]
+      -->
+      <xacro:homogeneous_inertia_definition
+        density="1000"
+        volume="0.00460251"
         center_of_mass="${[0.088782, -0.000001, 0.038098, 0, 0, 0]}"
         inertia_diagonal="${[0.00919, 0.08262, 0.08735]}"
@@ -185,5 +180,5 @@
           <origin xyz="0 0 0" rpy="0 0 0" />
           <geometry>
-            <mesh filename="package://puma560_description/meshes/puma_link_4.stl" />
+            <mesh filename="${puma_link_4_visual}" />
           </geometry>
           <material name="orange"/>
@@ -192,26 +187,19 @@
           <origin xyz="0 0 0" rpy="0 0 0" />
           <geometry>
-            <mesh filename="package://puma560_description/meshes/puma_link_4_collision.stl" />
-          </geometry>
-        </collision>
-      <!-- Inertia parameters
-      mass and center of mass (center_of_mass)
-      inertia_diagonal defined as [Ixx Iyy Izz]
-      inertia_off_diagonal defined as [Ixy Ixz Iyz]
-    -->
-    <!--     Parameters for uniform aluminium body -->
-    <xacro:general_inertia_definition
-      mass="1.27113"
-      center_of_mass="${[-0.000000, -0.000000, 0.047887, 0, 0, 0]}"
-      inertia_diagonal="${[0.00209, 0.00199, 0.00126]}"
-      inertia_off_diagonal="${[0, 0, 0]}"
-      />
-      <!--     Parameters for uniform generic body -->
-    <xacro:general_inertia_definition
-      mass="0.47079"
-      center_of_mass="${[-0.000000, -0.000000, 0.047887, 0, 0, 0]}"
-      inertia_diagonal="${[0.00077, 0.00074, 0.00047]}"
-      inertia_off_diagonal="${[0, 0, 0]}"
-      />
+            <mesh filename="${puma_link_4_collision}" />
+          </geometry>
+        </collision>
+      <!-- Create inertia matrix from parameters for homogeneous parts :
+      density[kg/m^3], volume[m^3] and center of mass[m]
+      inertia_diagonal defined as {Ixx Iyy Izz}[m^4]
+      inertia_off_diagonal defined as {Ixy Ixz Iyz}[m^4]
+      -->
+      <xacro:homogeneous_inertia_definition
+        density="1000"
+        volume="0.00047079"
+        center_of_mass="${[-0.000000, -0.000000, 0.047887, 0, 0, 0]}"
+        inertia_diagonal="${[0.00077, 0.00074, 0.00047]}"
+        inertia_off_diagonal="${[0, 0, 0]}"
+        />
       </link>
       <joint name="link_5" type="continuous">
@@ -225,5 +213,5 @@
           <origin xyz="0 0 0" rpy="0 0 0" />
           <geometry>
-            <mesh filename="package://puma560_description/meshes/puma_link_5.stl" />
+            <mesh filename="${puma_link_5_visual}" />
           </geometry>
           <material name="orange"/>
@@ -232,34 +220,19 @@
           <origin xyz="0 0 0" rpy="0 0 0" />
           <geometry>
-            <mesh filename="package://puma560_description/meshes/puma_link_5_collision.stl" />
-          </geometry>
-        </collision>
-      <!-- Inertia parameters
-      mass and center of mass (center_of_mass)
-      inertia_diagonal defined as [Ixx Iyy Izz]
-      inertia_off_diagonal defined as [Ixy Ixz Iyz]
-    -->
-    <!--     Parameters for uniform aluminium body -->
-    <xacro:general_inertia_definition
-      mass="0.20900"
-      center_of_mass="${[0.010974, 0.000000, 0.000000, 0, 0, 0]}"
-      inertia_diagonal="${[0.00005, 0.00012, 0.00012]}"
-      inertia_off_diagonal="${[0, 0, 0]}"
-      />
-      <!--     Parameters for uniform generic body -->
-    <xacro:general_inertia_definition
-      mass="0.07741"
-      center_of_mass="${[0.010974, 0.000000, 0.000000, 0, 0, 0]}"
-      inertia_diagonal="${[0.00002, 0.00004, 0.00005]}"
-      inertia_off_diagonal="${[0, 0, 0]}"
-      />
+            <mesh filename="${puma_link_5_collision}" />
+          </geometry>
+        </collision>
+      <!-- Create inertia matrix from parameters for homogeneous parts :
+      density[kg/m^3], volume[m^3] and center of mass[m]
+      inertia_diagonal defined as {Ixx Iyy Izz}[m^4]
+      inertia_off_diagonal defined as {Ixy Ixz Iyz}[m^4]
+      -->
+      <xacro:homogeneous_inertia_definition
+        density="1000"
+        volume="0.00007741"
+        center_of_mass="${[0.010974, 0.000000, 0.000000, 0, 0, 0]}"
+        inertia_diagonal="${[0.00002, 0.00004, 0.00005]}"
+        inertia_off_diagonal="${[0, 0, 0]}"
+        />
       </link>
     </robot>
-    <!--     Parameters for uniform body
-    <xacro:general_inertia_definition
-      mass="0"
-      center_of_mass="${[0, 0, 0, 0, 0, 0]}"
-      inertia_diagonal="${[0, 0, 0]}"
-      inertia_off_diagonal="${[0, 0, 0]}"
-      />
-    -->
