Commit message: MATLAB files added

File: puma560_description/urdf/puma560.xacro (robot description, xacro)
@@ -76,4 +76,5 @@
       <origin xyz="0 0 ${offset_z_link_1}" rpy="0 0 0" />
       <axis xyz="0 0 1" />
+      <dynamics damping="10.0" friction="0.0"/>
     </joint>
     <link name="puma_link_1">
@@ -109,4 +110,5 @@
       <origin xyz="0 ${offset_y_link_2} 0" rpy="${Pi/2} 0 0" />
       <axis xyz="0 0 1" />
+      <dynamics damping="1.0" friction="0.0"/>
     </joint>
     <link name="puma_link_2">
@@ -142,4 +144,5 @@
       <origin xyz="${offset_x_link_3} 0 0" rpy="0 0 0" />
       <axis xyz="0 0 1" />
+      <dynamics damping="0.0001" friction="0.0"/>
     </joint>
     <link name="puma_link_3">
@@ -175,4 +178,5 @@
       <origin xyz="${offset_x_link_4} 0 ${offset_z_link_4} " rpy="0 ${Pi/2} 0" />
       <axis xyz="0 0 1" />
+      <dynamics damping="0.0001" friction="0.0"/>
     </joint>
     <link name="puma_link_4">
@@ -208,4 +212,5 @@
       <origin xyz="0 0 ${offset_z_link_5} " rpy="0 ${-Pi/2} ${-Pi/2}" />
       <axis xyz="0 0 1" />
+      <dynamics damping="0.0001" friction="0.0"/>
     </joint>
     <link name="puma_link_5">
